File: 1_hardware_pcb/Main_Board_Loto/Main_Board_Loto.kicad_sch (KiCad schematic)
At the start: 66 parts, among them J2 V+-, J5 MOTOR_PINM1A, J6 MOTOR_PINM1B, J7 MOTOR_PINM1A, J8 MOTOR_PINM1B, Q1 2N7002, SW1 SW_SPST, SW2 START, SW3 START, U1 AMS1117-3.3, U10 QRE1113GR, U11 QRE1113GR, U12 QRE1113GR, U13 QRE1113GR, U15 ESP32_DevKit_V1_CH9102X, U2 LM7805_TO220, U3 TA6586, U5 TA6586, U6 QRE1113GR, U7 QRE1113GR, U8 QRE1113GR, U9 QRE1113GR

Commit message: SCH terminado
Parts:
- removed D3: LED, EESTN5-v2:Led_0805, symbol Device:LED
- removed R6: 220, EESTN5-v2:R_1206, symbol Device:R
- BZ1: footprint EESTN5-v2:Buzzer_12mm -> EESTN5:Buzzer_12mm
- C5: renamed from C7; footprint EESTN5-v2:C_0805 -> EESTN5:C_0805
- C9: footprint EESTN5-v2:C_0805 -> EESTN5:C_0805
- D1, D2: footprint EESTN5-v2:Led_0805 -> EESTN5:led_5mm_clear
- H1, H2, H3, H4, H5, H6: footprint EESTN5-v2:hole_3mm -> EESTN5:hole_3mm
- H7, H8: footprint EESTN5-v2:Separador_M3_5mm -> EESTN5:Separador_M3_5mm
- J1: renamed from J2; footprint EESTN5-v2:BORNERA2_AZUL -> EESTN5:BORNERA2_AZUL
- R1: renamed from R3; footprint EESTN5-v2:R_1206 -> EESTN5:R_1206
- R10: renamed from R13; footprint EESTN5-v2:R_0805 -> EESTN5:R_1206
- R11: renamed from R14; footprint EESTN5-v2:R_0805 -> EESTN5:R_1206
- R12: renamed from R15; footprint EESTN5-v2:R_0805 -> EESTN5:R_1206
- R13: renamed from R16; footprint EESTN5-v2:R_0805 -> EESTN5:R_1206
- R14: renamed from R17; footprint EESTN5-v2:R_0805 -> EESTN5:R_1206
- R15: renamed from R18; footprint EESTN5-v2:R_0805 -> EESTN5:R_1206
- R16: renamed from R19; footprint EESTN5-v2:R_0805 -> EESTN5:R_1206
- R17: renamed from R20; footprint EESTN5-v2:R_0805 -> EESTN5:R_1206
- R18: renamed from R21; footprint EESTN5-v2:R_0805 -> EESTN5:R_1206
- R19: renamed from R22; footprint EESTN5-v2:R_0805 -> EESTN5:R_1206
- R2: renamed from R5; footprint EESTN5-v2:R_1206 -> EESTN5:R_1206
- R20: renamed from R23; footprint EESTN5-v2:R_0805 -> EESTN5:R_1206
- R21: renamed from R24; footprint EESTN5-v2:R_0805 -> EESTN5:R_1206
- R3: renamed from R4; footprint EESTN5-v2:R_1206 -> EESTN5:R_1206
- R4: renamed from R8; footprint EESTN5-v2:R_1206 -> EESTN5:R_1206
- R5: renamed from R7; footprint EESTN5-v2:R_1206 -> EESTN5:R_1206
- R6: renamed from R9; footprint EESTN5-v2:R_0805 -> EESTN5:R_1206
- R7: renamed from R10; footprint EESTN5-v2:R_0805 -> EESTN5:R_1206
- R8: renamed from R11; footprint EESTN5-v2:R_0805 -> EESTN5:R_1206
- R9: renamed from R12; footprint EESTN5-v2:R_0805 -> EESTN5:R_1206
- SW2: renamed from SW1; footprint EESTN5-v2:SW_SPDT_TH_Vertical -> EESTN5:SW_SPDT_TH_Vertical
- U4: renamed from U15; footprint EESTN5-v2:ESP32_DevKit_V1_CH9102X -> EESTN5:ESP32_DevKit_V1_CH9102X
- renumbered C4 to C3, C5 to C4, C8 to C6, C11 to C7, C12 to C8, J5 to J2, J6 to J3, J7 to J4, J8 to J5, SW2 to SW1
Connections:
- net PUSH_1: now also U4.22 (TX2); no longer U4.21 (RX2)
- net PUSH_2: now also U4.21 (RX2); no longer U4.22 (TX2)
- net LED_BUILTING: no longer names the net of U4.19 (IO2)
Other:
- moved on the sheet: BZ1, D1, D2, Q1, R1, R3, R4
